File: Nucle-64-Template/Nucle64-template/Nucle64-template.kicad_pcb (KiCad board)
At the start: 2 copper layers, 70.3 x 84.6 mm, 2 parts, among them J1 Conn_02x19_Top_Bottom, J2 Conn_02x19_Top_Bottom

Commit message: Creación del digrama esquemático
Parts:
- added C1: 0.1µF, Capacitor_SMD:C_0805_2012Metric, F.Cu at (73.7, 8.08)
- added C2: 0.1µF, Capacitor_SMD:C_0805_2012Metric, F.Cu at (115.1, -16.7)
- added C3: 0.1µF, Capacitor_SMD:C_0805_2012Metric, F.Cu at (119.9, -22.3)
- added C4: 0.1µF, Capacitor_SMD:C_0805_2012Metric, F.Cu at (105.9, -7.61)
- added C5: 100nF, Capacitor_SMD:C_0805_2012Metric, F.Cu at (103.2, -4.66)
- added C6: 33nF, Capacitor_SMD:C_0805_2012Metric, F.Cu at (82.5, 8.79)
- added D1: LED, LED_THT:LED_D5.0mm, F.Cu at (89.9, -8.26)
- added D2: 1N4007, Diode_SMD:D_SOD-123, F.Cu at (83.9, -37.7)
- added D3: 1N4007, Diode_SMD:D_SOD-123, F.Cu at (78.2, -18.2)
- added D4: 1N4007, Diode_SMD:D_SOD-123, F.Cu at (83.9, -29.2)
- added D5: 1N4007, Diode_SMD:D_SOD-123, F.Cu at (60.4, -2.22)
- added D6: 1N4007, Diode_SMD:D_SOD-123, F.Cu at (83.9, -33.4)
- added J3: Screw_Terminal_01x03, Connector_Phoenix_MC:PhoenixContact_MCV_1,5_3-G-3.5_1x03_P3.50mm_Vertical, F.Cu at (165.5, 32.7)
- added J4: Screw_Terminal_01x02, Connector_Phoenix_MC:PhoenixContact_MCV_1,5_2-G-3.81_1x02_P3.81mm_Vertical, F.Cu at (44.5, 71.0)
- added J5: Screw_Terminal_01x02, Connector_Phoenix_MC:PhoenixContact_MCV_1,5_2-G-3.81_1x02_P3.81mm_Vertical, F.Cu at (46.5, 95.0)
- added J6: Conn_01x02_Male, Connector_PinHeader_2.54mm:PinHeader_1x02_P2.54mm_Vertical, F.Cu at (120.6, -37.5)
- added J7: Conn_01x02_Male, Connector_PinHeader_2.54mm:PinHeader_1x02_P2.54mm_Vertical, F.Cu at (110.0, -28.9)
- added Q1: 2N2219, Package_TO_SOT_SMD:SOT-23, F.Cu at (75.4, 1.13)
- added Q2: BTA16, Package_TO_SOT_THT:TO-220-3_Vertical, F.Cu at (137.5, 98.5)
- added R1: 1K5, Resistor_SMD:R_0805_2012Metric, F.Cu at (85.6, -3.01)
- added R10: 100R, Resistor_SMD:R_0805_2012Metric, F.Cu at (114.5, -26.8)
- added R11: 1K5, Resistor_SMD:R_0805_2012Metric, F.Cu at (85.6, 2.89)
- added R12: 1K5, Resistor_SMD:R_0805_2012Metric, F.Cu at (85.6, 5.84)
- added R13: 10k, Resistor_SMD:R_0805_2012Metric, F.Cu at (94.4, 2.89)
- added R14: 10k, Resistor_SMD:R_0805_2012Metric, F.Cu at (94.4, -3.01)
- added R15: 10k, Resistor_SMD:R_0805_2012Metric, F.Cu at (101.5, -10.6)
- added R16: 10k, Resistor_SMD:R_0805_2012Metric, F.Cu at (97.1, -7.61)
- added R17: 10K, Resistor_SMD:R_0805_2012Metric, F.Cu at (119.0, -28.2)
- added R18: 10K, Resistor_SMD:R_0805_2012Metric, F.Cu at (90.0, 2.89)
- added R19: 10k, Resistor_SMD:R_0805_2012Metric, F.Cu at (115.5, -23.9)
- added R2: 1K5, Resistor_SMD:R_0805_2012Metric, F.Cu at (97.1, -10.6)
- added R20: 10k, Resistor_SMD:R_0805_2012Metric, F.Cu at (110.7, -16.7)
- added R21: 100R, Resistor_SMD:R_0805_2012Metric, F.Cu at (101.5, -7.61)
- added R22: 100R, Resistor_SMD:R_0805_2012Metric, F.Cu at (115.1, -19.6)
- added R23: 1K, Resistor_SMD:R_0805_2012Metric, F.Cu at (105.9, -10.6)
- added R24: 47, Resistor_SMD:R_0805_2012Metric, F.Cu at (94.4, -0.06)
- added R25: 180R, Resistor_SMD:R_0805_2012Metric, F.Cu at (90.0, -0.06)
- added R26: 10k, Resistor_SMD:R_0805_2012Metric, F.Cu at (90.0, 5.84)
- added R27: 10k, Resistor_SMD:R_0805_2012Metric, F.Cu at (86.9, 8.79)
- added R28: 2k2, Resistor_SMD:R_0805_2012Metric, F.Cu at (98.8, -4.66)
- added R29: 33R, Resistor_SMD:R_0805_2012Metric, F.Cu at (110.7, -19.6)
- added R3: 100R, Resistor_SMD:R_0805_2012Metric, F.Cu at (90.0, -3.01)
- added R30: 100R, Resistor_SMD:R_0805_2012Metric, F.Cu at (98.8, -1.71)
- added R31: 10K, Resistor_SMD:R_0805_2012Metric, F.Cu at (110.7, -13.7)
- added R4: 100R, Resistor_SMD:R_0805_2012Metric, F.Cu at (85.6, -0.06)
- added R5: 100R, Resistor_SMD:R_0805_2012Metric, F.Cu at (78.1, 8.08)
- added R6: 100R, Resistor_SMD:R_0805_2012Metric, F.Cu at (114.5, -29.8)
- added R7: 100R, Resistor_SMD:R_0805_2012Metric, F.Cu at (106.6, -22.6)
- added R8: 100R, Resistor_SMD:R_0805_2012Metric, F.Cu at (120.4, -31.1)
- added R9: 100R, Resistor_SMD:R_0805_2012Metric, F.Cu at (111.0, -22.6)
- added RV1: 50K, Potentiometer_THT:Potentiometer_ACP_CA6-H2,5_Horizontal, F.Cu at (166.0, 41.0)
- added SW1: Rotary_Encoder_Switch, Rotary_Encoder:RotaryEncoder_Alps_EC12E-Switch_Vertical_H20mm_CircularMountingHoles, F.Cu at (187.5, 32.0)
- added SW2: SW_Push, Button_Switch_THT:SW_PUSH_6mm, F.Cu at (102.5, 22.0)
- added T1: 2SA798, User_models:2SA798, F.Cu at (101.9, -12.8)
- added T2: 2SA798, User_models:2SA798, F.Cu at (92.8, -12.8)
- added U1: DUY14A2, User_models:DUY14A2, F.Cu at (109.6, 39.1)
- added U2: DUY14A2, User_models:DUY14A2, F.Cu at (134.7, 39.2)
- added U3: 74HC14, Package_DIP:DIP-14_W7.62mm_Socket_LongPads, F.Cu at (77.5, 81.5)
- added U4: MOC3021M, Package_DIP:DIP-6_W10.16mm_LongPads, F.Cu at (34.2, 3.00)
- added U5: PC817, Package_DIP:DIP-4_W7.62mm, F.Cu at (61.5, 28.5)
- added U6: 74HC14, Package_DIP:DIP-14_W7.62mm_Socket_LongPads, F.Cu at (47.5, 55.5)
- added U7: TL081, Package_DIP:DIP-8_W7.62mm_Socket_LongPads, F.Cu at (75.5, 56.5)
